File: LFE5-Dev.kicad_sch (KiCad schematic)
At the start: 0 parts

Commit message: power and FT232H added
Parts:
- added C1, C10, C11, C13, C14, C18, C21, C3, C6, C7: 0u1, Capacitor_SMD:C_0603_1608Metric, symbol Device:C
- added C12, C19, C2, C20, C4, C5, C8, C9: 10u, Capacitor_SMD:C_0603_1608Metric, symbol Device:C
- added D1, D10, D11, D12, D2, D3, D4, D5, D6, D7, D8, D9: LED, LED_SMD:LED_0805_2012Metric, symbol Device:LED
- added FB1, FB2, FB3, FB4, FB5: FerriteBead, Inductor_SMD:L_0805_2012Metric, symbol Device:FerriteBead
- added FID1, FID2, FID3, FID4, FID5, FID6, FID7, FID8: Fiducial, Fiducial:Fiducial_1mm_Mask2mm, symbol Mechanical:Fiducial
- added J1: USB_C_Receptacle_USB2.0_14P, symbol Connector:USB_C_Receptacle_USB2.0_14P
- added L1, L2, L3: 2.2uH, Inductor_SMD:L_0805_2012Metric, symbol Device:L
- added R1, R12, R16, R17, R18, R19, R20, R21, R22, R23, R24, R25, R26, R27, R28, R5, R7, R8: 4k7 1%, Resistor_SMD:R_0603_1608Metric, symbol Device:R
- added R10: 500R 1%, Resistor_SMD:R_0603_1608Metric, symbol Device:R
- added R11: 6k8 1%, Resistor_SMD:R_0603_1608Metric, symbol Device:R
- added R13, R14, R4: 5k1 1%, Resistor_SMD:R_0603_1608Metric, symbol Device:R
- added R2, R9: 21k 1%, Resistor_SMD:R_0603_1608Metric, symbol Device:R
- added R3: 150R 1%, Resistor_SMD:R_0603_1608Metric, symbol Device:R
- added R6: 47k 1%, Resistor_SMD:R_0603_1608Metric, symbol Device:R
- added U1, U3, U4: TLV62568DBV, Package_TO_SOT_SMD:SOT-23-5, symbol Regulator_Switching:TLV62568DBV
- added U2: USBLC6-2SC6, Package_TO_SOT_SMD:SOT-23-6, symbol Power_Protection:USBLC6-2SC6
- added U6: TLV70225_SOT23-5, Package_TO_SOT_SMD:SOT-23-5, symbol Regulator_Linear:TLV70225_SOT23-5
Connections:
- new net: R4.1, R5.2, R6.2, U3.5 (FB)
- new net: J1.B5 (CC2), R13.1
- new net: D9.2 (A), R25.2
- new net: D4.2 (A), R20.2
- new net: D8.2 (A), R24.2
- new net: D2.2 (A), R18.2
- new net: L3.1, U4.3 (SW)
- new net: D1.2 (A), R17.2
- new net: C5.1, C6.1, FB4.2, R8.1, U4.4 (VIN)
- new net: R8.2, U4.1 (EN)
- new net: R10.2, R11.1, U4.5 (FB)
- new net: C10.1, C9.1, FB3.2, R1.1, U1.4 (VIN)
- new net: R1.2, U1.1 (EN)
- new net: C20.1, C21.1, FB5.2, R16.1, U6.1 (IN)
- new net: R7.2, U3.1 (EN)
- new net: L2.1, U3.3 (SW)
- new net: C1.1, C2.1, FB2.2, R7.1, U3.4 (VIN)
- new net: D7.2 (A), R23.2
- new net: D5.2 (A), R21.2
- new net: L1.1, U1.3 (SW)
- new net: R12.1, R3.2, U1.5 (FB)
- new net: R10.1, R9.2
- new net: C13.1, FB1.1, J1.A4 (VBUS), J1.A9 (VBUS), J1.B4 (VBUS), J1.B9 (VBUS), U2.5 (VBUS)
- new net: R16.2, U6.3 (EN)
- new net: D10.2 (A), R26.2
- new net: J1.A7 (D-), J1.B7 (D-), U2.1 (I/O1)
- new net: J1.A6 (D+), J1.B6 (D+), U2.3 (I/O2)
- new net: R2.2, R3.1
- new net: D6.2 (A), R22.2
- new net: D12.2 (A), R28.2
- new net: D3.2 (A), R19.2
- new net: J1.A5 (CC1), R14.1
- new net: D11.2 (A), R27.2
- new net +1V1: C3.1, C4.1, L2.2, R18.1, R5.1, R6.1
- new net +2V5: C18.1, C19.1, C7.1, C8.1, L3.2, R19.1, R9.1, U6.5 (OUT)
- new net +3V3: C11.1, C12.1, L1.2, R2.1, R20.1
- new net FT_D+: U2.4 (I/O2)
- new net FT_D-: U2.6 (I/O1)
- new net GND: C1.2, C10.2, C11.2, C12.2, C13.2, C14.2, C18.2, C19.2, C2.2, C20.2, C21.2, C3.2, C4.2, C5.2, C6.2, C7.2, C8.2, C9.2, D1.1 (K), D10.1 (K), D11.1 (K), D12.1 (K), D2.1 (K), D3.1 (K), D4.1 (K), D5.1 (K), D6.1 (K), D7.1 (K), D8.1 (K), D9.1 (K), J1.A1 (GND), J1.A12 (GND), J1.B1 (GND), J1.B12 (GND), J1.S1 (SHIELD), R11.2, R12.2, R13.2, R14.2, R4.2, U1.2 (GND), U2.2 (GND), U3.2 (GND), U4.2 (GND), U6.2 (GND)
- new net VBUS: C14.1, FB1.2, FB2.1, FB3.1, FB4.1, FB5.1, R17.1
Other:
- added sheet program and debug (program_debug.kicad_sch)
- note added: "Bottom:"
- note added: "Top:"
